File: actuator_driver.kicad_pcb (KiCad board)
At the start: 2 copper layers, 85.5 x 59 mm, 21 parts, among them J1 Conn_01x02_Pin, Q1 IRF540N, Q5 IRF540N, Q6 IRF540N, Q7 IRF540N, U1 FAN7389MX1

Commit message: connector update
Parts:
- added J2: Conn_01x07_Pin, Connector_JST:JST_EH_B7B-EH-A_1x07_P2.50mm_Vertical, F.Cu at (126.5, 100.5)
- added J3: Conn_01x02_Pin, TerminalBlock_WAGO:TerminalBlock_WAGO_236-102_1x02_P5.00mm_45Degree, F.Cu at (162.5, 97.5)
Connections:
- Q1 pad 3: unconnected-(Q1-S-Pad3) -> MOTOR1
