File: actuator_driver.kicad_sch (KiCad schematic)
At the start: 21 parts, among them J1 Conn_01x02_Pin, Q1 IRF540N, Q5 IRF540N, Q6 IRF540N, Q7 IRF540N, U1 FAN7389MX1

Commit message: other comp
Connections:
- net MOTOR1: now also Q1.3 (S)
Changed lines of the file:
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@@
 		(color 0 0 0 0)
 	)
+	(junction
+		(at 199.39 73.66)
+		(diameter 0)
+		(color 0 0 0 0)
+	)
 	(wire
 		(pts
@@
 		)
 		(stroke
+			(width 0)
+			(type default)
+		)
+	)
+	(wire
+		(pts
+			(xy 199.39 71.12) (xy 199.39 73.66)
+		)
+		(stroke

Commit message: connector update
Parts:
- added J2: Conn_01x07_Pin, Connector_JST:JST_EH_B7B-EH-A_1x07_P2.50mm_Vertical, symbol Connector:Conn_01x07_Pin
- added J3: Conn_01x02_Pin, TerminalBlock_WAGO:TerminalBlock_WAGO_236-102_1x02_P5.00mm_45Degree, symbol Connector:Conn_01x02_Pin
Connections:
- net +12V: now also J2.7 (Pin_7)
- net +48V: now also J3.1 (Pin_1)
- net EN_Driver: now also J2.1 (Pin_1)
- net GND: now also J2.6 (Pin_6), J3.2 (Pin_2)
- net HIN1: now also J2.5 (Pin_5)
- net HIN2: now also J2.4 (Pin_4)
- net LIN1: now also J2.3 (Pin_3)
- net LIN2: now also J2.2 (Pin_2)
